File: template/GameBoy_GamePak_AGB-002_Short/GameBoy_GamePak_AGB-002_Short.kicad_pcb (KiCad board)
At the start: 2 copper layers, 51 x 25.9 mm, 1 part, among them J1 GameBoy_GamePak_AGB-002

Commit message: Minor tweaks to footprints, updated templates accordingly
- Centered the footprint origins to improve ease of use
- Increased solder mask layers to outside the board outline for safety
- Updated templates with tweaked footprints
- Fixed typo in gitignore file
Parts:
- moved J1 27.2 mm to (149.6, 114.8)
